Commit message: feat: Add RTABMAP functionality
- Add RTABMAP and remap topics
- Created mapping and localization launch files
- Add compressed rtabmap.db file generated via robot teleop

File: Project_4/my_robot/urdf/my_robot.xacro (robot description, xacro)
@@ -118,4 +118,11 @@
     <dynamics damping="1.0" friction="1.0"/>
   </joint>
+  <joint name="camera_optical_joint" type="fixed">
+    <origin xyz="0 0 0" rpy="-1.5707 0 -1.5707"/>
+    <parent link="camera"/>
+    <child link="camera_link_optical"/>
+  </joint>
+  <link name="camera_link_optical">
+  </link>
   <!-- Optional -->
   <!-- <link name='right_wheel_f'>
